File: JLTT.kicad_pcb (KiCad board)
At the start: 2 copper layers, 68.6 x 53.3 mm, 23 parts, among them J1 Conn_01x03, J2 Conn_01x03, P1 Power, P2 Analog, P3 Digital, P4 Digital, P5 CONN_01X01, P6 CONN_01X01, P7 CONN_01X01, P8 CONN_01X01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

Commit message: PCB routing
Parts:
- C1, C2, C3, C4: footprint Capacitor_THT:CP_Axial_L10.0mm_D4.5mm_P15.00mm_Horizontal -> Capacitor_THT:CP_Radial_D4.0mm_P1.50mm
- R1, R2, R3, R4, R5: footprint Resistor_THT:R_Axial_DIN0309_L9.0mm_D3.2mm_P12.70mm_Horizontal -> Resistor_THT:R_Axial_DIN0207_L6.3mm_D2.5mm_P7.62mm_Horizontal
- moved J1 98.6 mm to (133.0, 98.4), turned to 90 degrees
- moved S1 95.5 mm to (131.0, 106.4)
- moved C2 88.2 mm to (171.0, 113.9), turned to 180 degrees
- moved C4 83.4 mm to (171.0, 98.9), turned to 180 degrees
- moved C3 82.6 mm to (153.5, 111.4)
- moved R1 81.8 mm to (148.5, 91.4), turned to 90 degrees
- moved J2 79.9 mm to (142.5, 105.9)
- moved C1 79.7 mm to (143.5, 91.4), turned to 90 degrees
- moved R3 78.5 mm to (171.0, 103.9), turned to 180 degrees
- moved BZ1 75.5 mm to (168.5, 81.4), turned to 270 degrees
- moved R4 62.5 mm to (138.5, 91.4), turned to 90 degrees
- moved R5 61.9 mm to (171.0, 108.9), turned to 180 degrees
- moved R2 58.7 mm to (153.5, 91.4), turned to 90 degrees
- moved RN24831 56.3 mm to (121.0, 108.9), turned to 90 degrees
- moved U1 49.7 mm to (156.0, 96.4), turned to 270 degrees
Connections:
- C4 pad 2: Net-(C4-Pad2) -> GND
- R2 pad 1: Net-(C4-Pad1) -> Net-(R2-Pad1)
- R3 pad 2: Net-(C4-Pad2) -> GND
- R5 pad 2: Net-(C4-Pad2) -> Net-(C4-Pad1)
- S1 pad 3: Net-(S1-Pad3) -> +5V
- S1 pad 8: Net-(S1-Pad8) -> GND
- U1 pad 2: Net-(C4-Pad1) -> Net-(R2-Pad1)
- U1 pad 6: Net-(C4-Pad2) -> Net-(C4-Pad1)
Routing:
- net +5V: track 0.00 -> 81.9 mm
- net /10: track 0.00 -> 55.6 mm
- net /11: track 0.00 -> 54.1 mm
- net Net-(C4-Pad1): track 0.00 -> 32.6 mm
- net /A1: track 0.00 -> 17.7 mm
- net /GasSelected1: track 0.00 -> 16.5 mm
- net Net-(C1-Pad1): track 0.00 -> 16.2 mm
- net /GasSensorLeft1: track 0.00 -> 12.2 mm
- net /GasSensorRight2: track 0.00 -> 11.2 mm
- net /GasSensorLeft2: track 0.00 -> 8.21 mm
- net /GasSensorRight1: track 0.00 -> 6.81 mm
- net /2: track 0.00 -> 6.18 mm
- net Net-(R2-Pad1): track 0.00 -> 5.02 mm
Other:
- board text added: "JLTT PCB iss 2019-2020"

Commit message: PCB copper gnd
Routing:
- added copper zone on B.Cu, net GND
Changed lines of the file:
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@@
   (segment (start 153.498 96.325) (end 153.458 96.365) (width 0.25) (layer B.Cu) (net 47))
   (segment (start 153.498 91.365) (end 153.498 96.325) (width 0.25) (layer B.Cu) (net 47))
+  (zone (net 4) (net_name GND) (layer B.Cu) (hatch edge 0.508)
+    (connect_pads (clearance 0.508))
+    (min_thickness 0.254)
+    (fill yes (arc_segments 32) (thermal_gap 0.508) (thermal_bridge_width 0.508))
+    (polygon
+      (pts
+        (xy 185.998 66.365) (xy 185.998 131.365) (xy 75.998 131.365) (xy 75.998 66.365)
+      )
+    )
+  )
 )
